File: pcb/ai_blinkle_16.brd (EAGLE design)
At the start: 44.5 x 44.5 mm, 24 parts

Commit message: routed
Parts:
- added DO: 1X01-SM, Ai_Connectors:1X01-SM
Connections:
- net DO: now also DO.1
Routing:
- net VCC: track 0.00 -> 131.7 mm
- net N$8: track 0.00 -> 12.5 mm, vias 0 -> 2
- net N$15: track 0.00 -> 12.5 mm, vias 0 -> 2
- net N$12: track 0.00 -> 12.5 mm, vias 0 -> 2
- net N$2: track 0.00 -> 12.5 mm, vias 0 -> 2
- net N$1: track 0.00 -> 12.5 mm, vias 0 -> 2
- net N$6: track 0.00 -> 12.5 mm, vias 0 -> 2
- net N$16: track 0.00 -> 12.5 mm, vias 0 -> 2
- net N$5: track 0.00 -> 12.5 mm, vias 0 -> 2
- net N$4: track 0.00 -> 12.5 mm, vias 0 -> 2
- net N$11: track 0.00 -> 12.5 mm, vias 0 -> 2
- net N$9: track 0.00 -> 12.5 mm, vias 0 -> 2
- net N$7: track 0.00 -> 12.5 mm, vias 0 -> 2
- net N$14: track 0.00 -> 12.5 mm, vias 0 -> 2
- net N$10: track 0.00 -> 12.4 mm, vias 0 -> 2
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
Commit message: done w version 1.0
Parts:
- added +, -, DI: 1X01-SM, Ai_Connectors:1X01-SM
- added LOGO: AI-LOGOXS, Ai_Miscellany:AI-LOGO-XS
Connections:
- net DI: now also DI.1
- net GND: now also -.1
- net VCC: now also +.1
Routing:
- net DI: track 0.00 -> 14.0 mm, vias 0 -> 1
- net VCC: track 131.7 -> 132.8 mm
- net N$1: vias 2 -> 3
Other:
- board text added: "+"
- board text added: "-"
- board text added: "BLINKLE 16"
- board text added: "DI"
- board text added: "DO"
- board text added: "Pasadena, CA"
- board text added: "www.acrobotic.com"
Changed lines of the file:
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@@
 <setting verticaltext="up"/>
 </settings>
-<grid distance="0.1" unitdist="mm" unit="mm" style="lines" multiple="1" display="yes" altdistance="0.025" altunitdist="inch" altunit="inch"/>
+<grid distance="5" unitdist="mil" unit="mil" style="lines" multiple="1" display="yes" altdistance="0.025" altunitdist="inch" altunit="inch"/>
 <layers>
 <layer number="1" name="Top" color="4" fill="1" visible="yes" active="yes"/>
@@
 <layer number="49" name="Reference" color="7" fill="1" visible="yes" active="yes"/>
 <layer number="50" name="dxf" color="7" fill="1" visible="no" active="no"/>
-<layer number="51" name="tDocu" color="7" fill="1" visible="yes" active="yes"/>
-<layer number="52" name="bDocu" color="7" fill="1" visible="yes" active="yes"/>
+<layer number="51" name="tDocu" color="7" fill="1" visible="no" active="yes"/>
+<layer number="52" name="bDocu" color="7" fill="1" visible="no" active="yes"/>
 <layer number="53" name="tGND_GNDA" color="7" fill="9" visible="no" active="no"/>
 <layer number="54" name="bGND_GNDA" color="1" fill="9" visible="no" active="no"/>
@@
 <circle x="22.225" y="22.225" radius="22.225" width="0.127" layer="20"/>
 <circle x="22.225" y="22.225" radius="15.875" width="0.127" layer="20"/>
+<text x="30.648" y="36.9694" size="0.762" layer="22" font="vector" ratio="15" rot="MR11.2">www.acrobotic.com</text>
+<text x="18.9894" y="42.8114" size="1.016" layer="22" font="vector" ratio="15" rot="MR348.7">DO</text>
+<text x="34.4834" y="39.0014" size="1.016" layer="22" font="vector" ratio="15" rot="MR33.7">DI</text>
+<text x="10.1444" y="5.3724" size="1.27" layer="22" font="vector" ratio="15" rot="MR213.7">+</text>
+<text x="26.838" y="0.6982" size="1.27" layer="22" font="vector" ratio="15" rot="MR348.7">-</text>
+<text x="5.121" y="24.9044" size="0.762" layer="22" font="vector" ratio="15" rot="MR112.5">BLINKLE 16</text>
+<text x="26.1776" y="5.4226" size="0.762" layer="22" font="vector" ratio="15" rot="MR0">Pasadena, CA</text>
 </plain>
 <attributes>
@@
 <element name="C7" library="Ai_Passives" package="CAP-0402" value="0.1uF" x="2.286" y="26.1874" smashed="yes" rot="R168.8"/>
 <element name="C8" library="Ai_Passives" package="CAP-0402" value="0.1uF" x="10.9474" y="39.116" smashed="yes" rot="R123.8"/>
-<element name="DO" library="Ai_Connectors" package="1X01-SM" value="1X01-SM" x="18.375" y="41.625" smashed="yes">
-<attribute name="NAME" x="18.995" y="43.851" size="1.016" layer="25" font="vector" ratio="15" rot="R191.3"/>
+<element name="DO" library="Ai_Connectors" package="1X01-SM" value="1X01-SM" x="18.3642" y="41.6306" smashed="yes">
+<attribute name="NAME" x="18.9842" y="43.8566" size="1.016" layer="25" font="vector" ratio="15" rot="R191.3"/>
 </element>
+<element name="DI" library="Ai_Connectors" package="1X01-SM" value="1X01-SM" x="33.2232" y="38.6588" smashed="yes">
+<attribute name="NAME" x="33.3532" y="39.7828" size="1.016" layer="25" font="vector" ratio="15" rot="R326.3"/>
+</element>
+<element name="+" library="Ai_Connectors" package="1X01-SM" value="1X01-SM" x="11.2268" y="5.7912" smashed="yes">
+<attribute name="NAME" x="10.6568" y="3.7152" size="1.27" layer="25" font="vector" ratio="15" rot="SR56.3"/>
+</element>
+<element name="-" library="Ai_Connectors" package="1X01-SM" value="1X01-SM" x="26.0858" y="2.8194" smashed="yes" rot="R191.3">
+<attribute name="NAME" x="26.8298" y="1.97379375" size="1.27" layer="25" font="vector" ratio="15" rot="R191.3"/>
+</element>
+<element name="LOGO" library="Ai_Miscellany" package="AI-LOGO-XS" value="AI-LOGOXS" x="27.05" y="39.8" rot="MR11.2"/>
 </elements>
 <signals>
@@
 <wire x1="38.374003125" y1="9.1872625" x2="36.45413125" y2="9.1872625" width="0.254" layer="1"/>
 <wire x1="36.45413125" y1="9.1872625" x2="33.14100625" y2="5.8741375" width="0.254" layer="1"/>
-<wire x1="24.425" y1="1.575" x2="23.07638125" y2="2.92361875" width="0.254" layer="1"/>
+<wire x1="24.425" y1="1.575" x2="23.8" y2="2.2" width="0.254" layer="1"/>
+<wire x1="23.8" y1="2.2" x2="23.07638125" y2="2.92361875" width="0.254" layer="1"/>
 <wire x1="23.07638125" y1="2.92361875" x2="18.38885" y2="2.92361875" width="0.254" layer="1"/>
 <wire x1="9.1872625" y1="6.07599375" x2="9.1872625" y2="7.995865625" width="0.254" layer="1"/>
 <wire x1="9.1872625" y1="7.995865625" x2="5.8741375" y2="11.308990625" width="0.254" layer="1"/>
 <wire x1="12.29036875" y1="40.463503125" x2="18.863503125" y2="40.463503125" width="0.254" layer="1"/>
-<wire x1="28.09455625" y1="42.147309375" x2="31.8678625" y2="38.374003125" width="0.254" layer="1"/>
-<wire x1="31.8678625" y1="38.374003125" x2="35.262734375" y2="38.374003125" width="0.254" layer="1"/>
 <wire x1="40.463503125" y1="32.159628125" x2="40.463503125" y2="26.836496875" width="0.254" layer="1"/>
 <wire x1="40.463503125" y1="26.836496875" x2="42.875" y2="24.425" width="0.254" layer="1"/>
 <wire x1="42.147309375" y1="16.355440625" x2="38.374003125" y2="12.582134375" width="0.254" layer="1"/>
 <wire x1="38.374003125" y1="12.582134375" x2="38.374003125" y2="9.1872625" width="0.254" layer="1"/>
-<wire x1="32.159628125" y1="3.98649375" x2="26.83649375" y2="3.98649375" width="0.254" layer="1"/>
-<wire x1="26.83649375" y1="3.98649375" x2="24.425" y2="1.575" width="0.254" layer="1"/>
-<wire x1="16.355440625" y1="2.3026875" x2="12.582134375" y2="6.07599375" width="0.254" layer="1"/>
-<wire x1="12.582134375" y1="6.07599375" x2="9.1872625" y2="6.07599375" width="0.254" layer="1"/>
+<wire x1="32.159628125" y1="3.98649375" x2="25.58649375" y2="3.98649375" width="0.254" layer="1"/>
+<wire x1="16.355440625" y1="2.3026875" x2="13.232134375" y2="5.52599375" width="0.254" layer="1"/>
 <wire x1="1.575" y1="20.025" x2="2.92361875" y2="21.37361875" width="0.254" layer="1"/>
 <wire x1="2.92361875" y1="21.37361875" x2="2.92361875" y2="26.061146875" width="0.254" layer="1"/>
@@
 <wire x1="6.07599375" y1="35.262734375" x2="7.995865625" y2="35.262734375" width="0.254" layer="1"/>
 <wire x1="7.995865625" y1="35.262734375" x2="11.308990625" y2="38.575859375" width="0.254" layer="1"/>
+<contactref element="+" pad="1"/>
 <wire x1="18.863503125" y1="40.463503125" x2="20.65" y2="42.25" width="0.254" layer="1"/>
-<wire x1="4.892759375" y1="12.29036875" x2="3.98649375" y2="12.29036875" width="0" layer="19" extent="1-1"/>
+<wire x1="25.58649375" y1="3.98649375" x2="23.8" y2="2.2" width="0.254" layer="1"/>
+<wire x1="13.232134375" y1="5.52599375" x2="11.2268" y2="5.7912" width="0.254" layer="1"/>
+<wire x1="11.2268" y1="5.7912" x2="9.1872625" y2="6.07599375" width="0.254" layer="1"/>
+<wire x1="3.98649375" y1="12.29036875" x2="3.98649375" y2="17.61350625" width="0.254" layer="1"/>
+<wire x1="3.98649375" y1="17.61350625" x2="1.575" y2="20.025" width="0.254" layer="1"/>
+<wire x1="3.98649375" y1="12.29036875" x2="4.892759375" y2="12.29036875" width="0.254" layer="1"/>
 </signal>
 <signal name="GND">
@@
 <contactref element="C8" pad="2"/>
 <contactref element="C6" pad="2"/>
+<contactref element="-" pad="1"/>
+<via x="15.6718" y="4.6482" extent="1-16" drill="0.381"/>
 </signal>
 <signal name="N$1">
@@
 <wire x1="20.05" y1="39.7" x2="22.2" y2="39.7" width="0.254" layer="1"/>
 <via x="22.2" y="39.7" extent="1-16" drill="0.381"/>
-<wire x1="22.2" y1="39.7" x2="30.2" y2="41.3" width="0.254" layer="16"/>
-<via x="30.2" y="41.3" extent="1-16" drill="0.381"/>
-<wire x1="30.2" y1="41.3" x2="32.159628125" y2="40.463503125" width="0.254" layer="1"/>
+<via x="30.4" y="41.25" extent="1-16" drill="0.381"/>
+<wire x1="30.4" y1="41.25" x2="32.159628125" y2="40.463503125" width="0.254" layer="1"/>
+<via x="27.8" y="40.75" extent="1-16" drill="0.381"/>
+<wire x1="30.4" y1="41.25" x2="27.8" y2="40.75" width="0.254" layer="1"/>
+<wire x1="22.2" y1="39.7" x2="27.8" y2="40.75" width="0.254" layer="16"/>
 </signal>
 <signal name="N$2">
@@
 <wire x1="26.86996875" y1="39.19089375" x2="28.829" y2="38.354" width="0.254" layer="1"/>
 <via x="28.829" y="38.354" extent="1-16" drill="0.381"/>
-<wire x1="28.829" y1="38.354" x2="36.83" y2="36.83" width="0.254" layer="16"/>
-<via x="36.83" y="36.83" extent="1-16" drill="0.381"/>
-<wire x1="36.83" y1="36.83" x2="38.374003125" y2="35.262734375" width="0.254" layer="1"/>
+<wire x1="28.829" y1="38.354" x2="36.93" y2="36.73" width="0.254" layer="16"/>
+<via x="36.93" y="36.73" extent="1-16" drill="0.381"/>
+<wire x1="36.93" y1="36.73" x2="38.374003125" y2="35.262734375" width="0.254" layer="1"/>
 </signal>
 <signal name="DI">
 <contactref element="LED1" pad="4"/>
+<contactref element="DI" pad="1"/>
+<wire x1="24.425" y1="42.875" x2="22.39" y2="42.88" width="0.254" layer="1"/>
+<via x="22.39" y="42.88" extent="1-16" drill="0.381"/>
+<wire x1="22.39" y1="42.88" x2="26" y2="42.9" width="0.254" layer="16"/>
+<wire x1="26" y1="42.9" x2="33.2232" y2="38.6588" width="0.254" layer="16"/>
 </signal>
 <signal name="N$4">
@@
 <contactref element="LED10" pad="2"/>
 <contactref element="LED11" pad="4"/>
-<wire x1="17.580028125" y1="5.259103125" x2="15.8" y2="6" width="0.254" layer="1"/>
-<via x="15.8" y="6" extent="1-16" drill="0.381"/>
-<wire x1="15.8" y1="6" x2="7.5" y2="7.7" width="0.254" layer="16"/>
+<wire x1="17.580028125" y1="5.259103125" x2="15.5206" y2="6.1524" width="0.254" layer="1"/>
+<via x="15.5206" y="6.1524" extent="1-16" drill="0.381"/>
+<wire x1="15.5206" y1="6.1524" x2="7.5" y2="7.7" width="0.254" layer="16"/>
 <via x="7.5" y="7.7" extent="1-16" drill="0.381"/>
 <wire x1="7.5" y1="7.7" x2="6.07599375" y2="9.1872625" width="0.254" layer="1"/>
@@
 <wire x1="13.51495625" y1="37.5070875" x2="15.6" y2="38.4" width="0.254" layer="1"/>
 <via x="15.6" y="38.4" extent="1-16" drill="0.381"/>
-<wire x1="15.6" y1="38.4" x2="18.375" y2="41.625" width="0.254" layer="16"/>
+<wire x1="15.6" y1="38.4" x2="18.3642" y2="41.6306" width="0.254" layer="16"/>
 </signal>
 </signals>
