File: pcb/ai_blinkle_16.sch (EAGLE design)
At the start: 24 parts

Commit message: routed
Parts:
- added DO: 1X01-SM, Ai_Connectors:1X01-SM
Connections:
- net DO: now also DO.1
Changed lines of the file:
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@@
 <part name="C7" library="Ai_Passives" deviceset="CAP" device="0402" value="0.1uF"/>
 <part name="C8" library="Ai_Passives" deviceset="CAP" device="0402" value="0.1uF"/>
+<part name="DO" library="Ai_Connectors" deviceset="1X01" device="-SM" value="1X01-SM"/>
 </parts>
 <sheets>
@@
 <instance part="C7" gate="G$1" x="132.08" y="167.64"/>
 <instance part="C8" gate="G$1" x="137.16" y="167.64"/>
+<instance part="DO" gate="G$1" x="104.14" y="146.05"/>
 </instances>
 <busses>
@@
 <label x="53.34" y="162.56" size="1.27" layer="95" font="vector" ratio="15" rot="R180" xref="yes"/>
 </segment>
-</net>
+<segment>
+<pinref part="DO" gate="G$1" pin="1"/>
+<wire x1="109.22" y1="146.05" x2="111.76" y2="146.05" width="0.1524" layer="91"/>
+<label x="111.76" y="146.05" size="1.27" layer="95" font="vector" ratio="15" xref="yes"/>
+</segment>
+</net>

Commit message: done w version 1.0
Parts:
- added +, -, DI: 1X01-SM, Ai_Connectors:1X01-SM
- added LOGO: AI-LOGOXS, Ai_Miscellany:AI-LOGOXS
Connections:
- net DI: now also DI.1
- net GND: now also -.1
- net VCC: now also +.1
Changed lines of the file:
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@@
 <part name="C8" library="Ai_Passives" deviceset="CAP" device="0402" value="0.1uF"/>
 <part name="DO" library="Ai_Connectors" deviceset="1X01" device="-SM" value="1X01-SM"/>
+<part name="DI" library="Ai_Connectors" deviceset="1X01" device="-SM" value="1X01-SM"/>
+<part name="+" library="Ai_Connectors" deviceset="1X01" device="-SM" value="1X01-SM"/>
+<part name="-" library="Ai_Connectors" deviceset="1X01" device="-SM" value="1X01-SM"/>
+<part name="LOGO" library="Ai_Miscellany" deviceset="AI-LOGO" device="XS"/>
 </parts>
 <sheets>
@@
 <instance part="C8" gate="G$1" x="137.16" y="167.64"/>
 <instance part="DO" gate="G$1" x="104.14" y="146.05"/>
+<instance part="DI" gate="G$1" x="104.14" y="137.16"/>
+<instance part="+" gate="G$1" x="104.14" y="128.27"/>
+<instance part="-" gate="G$1" x="104.14" y="119.38"/>
+<instance part="LOGO" gate="G$1" x="138.43" y="12.7"/>
 </instances>
 <busses>
@@
 <junction x="121.92" y="173.99"/>
 </segment>
+<segment>
+<pinref part="+" gate="G$1" pin="1"/>
+<wire x1="109.22" y1="128.27" x2="111.76" y2="128.27" width="0.1524" layer="91"/>
+<label x="111.76" y="128.27" size="1.27" layer="95" font="vector" ratio="15" xref="yes"/>
+</segment>
 </net>
 <net name="GND" class="0">
@@
 <junction x="121.92" y="161.29"/>
 </segment>
+<segment>
+<pinref part="-" gate="G$1" pin="1"/>
+<wire x1="109.22" y1="119.38" x2="111.76" y2="119.38" width="0.1524" layer="91"/>
+<label x="111.76" y="119.38" size="1.27" layer="95" font="vector" ratio="15" xref="yes"/>
+</segment>
 </net>
 <net name="N$1" class="0">
@@
 <label x="44.45" y="170.18" size="1.27" layer="95" font="vector" ratio="15" xref="yes"/>
 </segment>
-</net>
+<segment>
+<pinref part="DI" gate="G$1" pin="1"/>
+<wire x1="109.22" y1="137.16" x2="111.76" y2="137.16" width="0.1524" layer="91"/>
+<label x="111.76" y="137.16" size="1.27" layer="95" font="vector" ratio="15" xref="yes"/>
+</segment>
+</net>
