File: pcb/ai_aureola-16.brd (EAGLE design)
At the start: 44.5 x 44.5 mm, 29 parts

Commit message: ready for manufacturing
Parts:
- added R1: 300, Ai_Passives:RES-0402
- moved DO 15.1 mm to (5.77, 33.2)
Connections:
- new net N$3: DI.1, R1.2
- net DI: now also R1.1; no longer DI.1
Routing:
- net N$3: track 0.00 -> 15.3 mm
- net DI: track 14.0 -> 11.0 mm
- net DO: track 6.52 -> 9.32 mm, vias 1 -> 0
- net VCC: track 132.8 -> 134.0 mm, vias 0 -> 2
Other:
- board text added: "AUREOLA-16"
- board text removed: "BLINKLE 16"
